File: 12bitbadge.sch (KiCad schematic (older format))
At the start: 47 parts, among them J1 Conn_02x04_Counter_Clockwise, J2 Conn_02x04_Counter_Clockwise, J3 Conn_02x04_Counter_Clockwise, J4 Conn_02x03_Odd_Even, J5 Conn_02x03_Odd_Even, J6 Conn_02x03_Odd_Even, J7 Conn_02x03_Odd_Even, Q1 Q_PMOS_GSD, Q2 Q_PMOS_GSD, Q3 Q_PMOS_GSD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

Commit message: Redesigning as a through-hole kit
Parts:
- removed J1, J2, J3: Conn_02x04_Counter_Clockwise, 12bitbadge:SOIC_clipProgSmall, symbol Connector_Generic:Conn_02x04_Counter_Clockwise
- removed J6, J7: Conn_02x03_Odd_Even, Connector_PinSocket_2.54mm:PinSocket_2x03_P2.54mm_Vertical, symbol Connector_Generic:Conn_02x03_Odd_Even
- removed R9: 200k, Resistor_SMD:R_0805_2012Metric_Pad1.15x1.40mm_HandSolder, symbol Device:R
- removed SW10, SW11, SW12, SW2, SW3, SW4, SW5, SW6, SW7, SW8, SW9: SW_SPDT, Button_Switch_THT:SW_CuK_JS202011CQN_DPDT_Straight, symbol Switch:SW_SPDT
- removed U1, U2, U3: ATtiny10-TS, Package_TO_SOT_SMD:SOT-23-6_Handsoldering, symbol MCU_Microchip_ATtiny:ATtiny10-TS
- added C?: C, symbol Device:C
- added C?: 10nF, symbol Device:C
- added J2, J3: Conn_02x03_Odd_Even, Connector_PinSocket_2.54mm:PinSocket_2x03_P2.54mm_Vertical, symbol Connector_Generic:Conn_02x03_Odd_Even
- added J?: Conn_02x03_Odd_Even, Connector_PinHeader_2.54mm:PinHeader_2x03_P2.54mm_Vertical, symbol Connector_Generic:Conn_02x03_Odd_Even
- added Q?: Q_PMOS_GSD, Package_TO_SOT_SMD:SOT-23_Handsoldering, symbol Device:Q_PMOS_GSD
- added R16, R25, R? (x2): 100k, Resistor_SMD:R_0805_2012Metric_Pad1.15x1.40mm_HandSolder, symbol Device:R
- added R17, R22, R26: 200k, Resistor_SMD:R_0805_2012Metric_Pad1.15x1.40mm_HandSolder, symbol Device:R
- added R18, R27, R?: 1k, Resistor_SMD:R_0805_2012Metric_Pad1.15x1.40mm_HandSolder, symbol Device:R
- added R19, R23: 25k, Resistor_SMD:R_0805_2012Metric_Pad1.15x1.40mm_HandSolder, symbol Device:R
- added R24: 50k, Resistor_SMD:R_0805_2012Metric_Pad1.15x1.40mm_HandSolder, symbol Device:R
- added RV?: 100kΩ, symbol Device:R_POT
- added SW10, SW11, SW12, SW2, SW3, SW4, SW5, SW6, SW7, SW8, SW9: SW_SPDT, Button_Switch_THT:SW_CuK_JS202011CQN_DPDT_Straight, symbol Switch:SW_Push_DPDT
- added U?: TLC555CP, symbol Timer:TLC555CP
- added U?: ATtiny85-20PU, Package_DIP:DIP-8_W7.62mm, symbol MCU_Microchip_ATtiny:ATtiny85-20PU
- R11, R15, R6: value 25k -> 50k
- R12, R7: value 50k -> 100k
- R13, R8: value 100k -> 200k
- R14: value 200k -> 25k
- R20: value 1k -> 50k
- R21: value 1k -> 100k
- SW1: symbol Switch:SW_SPDT -> Switch:SW_Push_DPDT
- renumbered J5 to J1, R16 to R28, R17 to R29, R18 to R30, R19 to R9
Connections:
- net 0V: now also SW1.5 (B), C?.1, J2.2 (Pin_2), J3.2 (Pin_2), R?.1, RV?.3, SW5.5 (B), SW9.5 (B), U?.1 (GND), U?.4 (GND); no longer R10.1, R15.1, R5.1
- net 3.3V: now also Q?.3 (D), SW5.2 (B), SW9.2 (B), U?.8 (VCC)
- net ADC_1: now also R13.1, R8.1, R17.1, R22.1, R26.1, SW12.3 (C), SW12.4 (A), SW4.3 (C), SW4.4 (A), SW8.3 (C), SW8.4 (A); no longer R5.2
- net PWR_OUT_2: now also J2.1 (Pin_1)
- net PWR_OUT_3: now also J3.1 (Pin_1)
- net R_OUT: now also R18.2, R27.2
- net at R2.1: now also SW2.3 (C), SW3.2 (B)
- net at R2.2: now also SW2.1 (A)
- net at R3.2: now also SW3.1 (A)
- net at R3.1: now also SW3.3 (C), SW4.2 (B)
- net at R4.2: now also SW4.1 (A)
- net at R1.1, SW1.3 (C): now also SW2.2 (B)
- net at R7.1: now also SW3.4 (A), SW4.5 (B)
- net at R7.2: now also SW3.6 (C)
- net at R8.2: now also SW4.6 (C)
- net at R6.1: now also SW2.4 (A), SW3.5 (B)
- net at R6.2: now also SW2.6 (C)
- net at R12.1: now also SW7.3 (C), SW8.2 (B)
- net at R12.2: now also SW7.1 (A)
- net at R13.2: now also SW8.1 (A)
- net at R14.2: now also SW5.6 (C)
- net at R11.1: now also SW6.3 (C), SW7.2 (B)
- net at R11.2: now also SW6.1 (A)
- net at Q2.1 (G): now also R18.1; no longer R20.1
- net at R21.1: now also SW11.3 (C), SW12.2 (B); no longer Q3.1 (G)
- net ADC_2: no longer names the net of R10.2
- net ADC_2: now also SW5.1 (A)
- net ADC_3: no longer names the net of R14.1
- net ADC_3: now also SW5.4 (A), SW6.5 (B); no longer R15.2
- net B_OUT: no longer names the net of R21.2
- net B_OUT: now also SW11.1 (A)
- net G_OUT: no longer names the net of R20.2
- net G_OUT: now also SW10.1 (A)
- new net: R5.1, SW1.4 (A), SW2.5 (B)
- new net: R5.2, SW1.6 (C)
- new net: R10.1, SW5.3 (C), SW6.2 (B)
- new net: R15.1, SW6.4 (A), SW7.5 (B)
- new net: R15.2, SW6.6 (C)
- new net: R16.1, SW7.4 (A), SW8.5 (B)
- new net: R16.2, SW7.6 (C)
- new net: R17.2, SW8.6 (C)
- new net: R20.1, SW10.3 (C), SW11.2 (B)
- new net: R22.2, SW12.1 (A)
- new net: R19.1, SW10.2 (B), SW9.3 (C)
- new net: R19.2, SW9.1 (A)
- new net: R23.1, SW10.5 (B), SW9.4 (A)
- new net: R23.2, SW9.6 (C)
- new net: Q3.1 (G), R27.1
- new net: R24.1, SW10.4 (A), SW11.5 (B)
- new net: R24.2, SW10.6 (C)
- new net: R25.1, SW11.4 (A), SW12.5 (B)
- new net: R25.2, SW11.6 (C)
- new net: R26.2, SW12.6 (C)
- new net: C?.1, R?.1, R?.2, U?.2 (TR), U?.6 (THR)
- new net: R?.2, U?.3 (Q)
- new net: C?.2, U?.5 (CV)
- new net: C?.2, RV?.2
- new net: Q?.1 (G), R?.1
- new net PWR_IN: Q?.2 (S), R?.2, RV?.1, U?.4 (R), U?.8 (VCC)
Other:
- moved on the sheet: J1, Q1, R9
