File: 12bitbadge.sch (KiCad schematic (older format))
At the start: 60 parts, among them J1 Conn_02x03_Odd_Even, J2 Conn_02x03_Odd_Even, J3 Conn_02x03_Odd_Even, J4 Conn_02x03_Odd_Even, Q1 Q_PMOS_GSD, Q2 Q_PMOS_GSD, Q3 Q_PMOS_GSD, SW1 SW_SPDT, SW10 SW_SPDT, SW11 SW_SPDT, SW12 SW_SPDT, SW2 SW_SPDT, SW3 SW_SPDT, SW4 SW_SPDT, SW5 SW_SPDT, SW6 SW_SPDT, SW7 SW_SPDT, SW8 SW_SPDT, SW9 SW_SPDT

Commit message: Continued work on kit version
Parts:
- removed Q1, Q2, Q3: Q_PMOS_GSD, Package_TO_SOT_SMD:SOT-23_Handsoldering, symbol Device:Q_PMOS_GSD
- added Q1, Q2, Q3: Q_PMOS_GDS, Package_TO_SOT_SMD:TO-252-2, symbol Device:Q_PMOS_GDS
- C1: renamed from C?; value C -> 10 nF; footprint (none) -> Capacitor_THT:C_Disc_D4.3mm_W1.9mm_P5.00mm
- C2: renamed from C?; footprint (none) -> Capacitor_THT:C_Disc_D4.3mm_W1.9mm_P5.00mm
- Q4: renamed from Q?; value Q_PMOS_GSD -> Q_PMOS_GDS; footprint Package_TO_SOT_SMD:SOT-23_Handsoldering -> Package_TO_SOT_SMD:TO-252-2; symbol Device:Q_PMOS_GSD -> Device:Q_PMOS_GDS
- R1, R10, R11, R12, R13, R14, R15, R16, R17, R18, R19, R2, R20, R21, R22, R23, R24, R25, R26, R27, R28, R29, R3, R30, R4, R5, R6, R7, R8, R9: footprint Resistor_SMD:R_0805_2012Metric_Pad1.15x1.40mm_HandSolder -> Resistor_THT:R_Axial_DIN0204_L3.6mm_D1.6mm_P5.08mm_Horizontal
- R31, R32, R33: renamed from R?; footprint Resistor_SMD:R_0805_2012Metric_Pad1.15x1.40mm_HandSolder -> Resistor_THT:R_Axial_DIN0204_L3.6mm_D1.6mm_P5.08mm_Horizontal
- RV1: renamed from RV?; footprint (none) -> Potentiometer_THT:Potentiometer_Alpha_RD901F-40-00D_Single_Vertical_CircularHoles
- U1: renamed from U?; footprint (none) -> Package_DIP:DIP-8_W7.62mm
- gave numbers to parts that had none: 2
Connections:
- net 0V: now also J5.6 (Pin_6)
- net 3.3V: now also J5.2 (Pin_2), Q4.2 (D), Q1.3 (S), Q2.3 (S), Q3.3 (S); no longer J4.1 (Pin_1), Q4.3 (D)
- net ADC_1: now also J5.5 (Pin_5), U2.1 (~RESET~/PB5); no longer R13.1, R17.1, R22.1, R26.1, SW12.3 (C), SW12.4 (A), SW8.3 (C), SW8.4 (A)
- net PWR_IN: now also J4.1 (Pin_1), Q4.3 (S); no longer Q4.2 (S)
- net PWR_OUT_1: now also Q1.2 (D)
- net PWR_OUT_2: now also Q2.2 (D)
- net PWR_OUT_3: now also Q3.2 (D)
- net R_OUT: now also J5.3 (Pin_3), U2.7 (PB2); no longer R18.2, R27.2
- net at R9.1: now also Q1.1 (G)
- net at R18.1: now also Q2.1 (G)
- net at R27.1: now also Q3.1 (G)
- net ADC_2: now reaches U2.2 (XTAL1/PB3)
- net ADC_2: now also R13.1, R17.1, SW8.3 (C), SW8.4 (A)
- net ADC_3: now reaches U2.3 (XTAL2/PB4)
- net ADC_3: now also R22.1, R26.1, SW12.3 (C), SW12.4 (A)
- net B_OUT: now reaches U2.5 (AREF/PB0)
- net B_OUT: now also J5.4 (Pin_4), R27.2
- net G_OUT: now reaches U2.6 (PB1)
- net G_OUT: now also J5.1 (Pin_1), R18.2
