File: 12bitbadge.kicad_pcb (KiCad board)
At the start: 2 copper layers, 62.6 x 53.7 mm, 47 parts, among them J1 Conn_02x04_Counter_Clockwise, J2 Conn_02x04_Counter_Clockwise, J3 Conn_02x04_Counter_Clockwise, J4 Conn_02x03_Odd_Even, J5 Conn_02x03_Odd_Even, J6 Conn_02x03_Odd_Even, J7 Conn_02x03_Odd_Even, Q1 Q_PMOS_GSD, Q2 Q_PMOS_GSD, Q3 Q_PMOS_GSD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

Commit message: Changed from common-anode RGB LED to common-cathode RGB LED
Parts:
- D1: value LED_RAGB -> LED_RCGB
- R1, R11, R6: value 25k -> 200k
- R12, R2, R7: value 50k -> 100k
- R13, R3, R8: value 100k -> 50k
- R14, R4, R9: value 200k -> 25k
- moved D1 3.81 mm to (141.7, 61.6), turned to 270 degrees
Connections:
- D1 pad 2: 3.3V -> 0V
- R16 pad 2: Net-(D1-Pad4) -> Net-(D1-Pad1)
- R18 pad 2: Net-(D1-Pad1) -> Net-(D1-Pad4)
Routing:
- net 0V: track 156.3 -> 225.5 mm
- net 3.3V: track 154.8 -> 140.0 mm
